Commit message: 重建proto，易于标定零点

File: DogURDF/dog_asm2/urdf/dog_asm2.urdf (robot description, URDF)
Before this commit: robot dog_asm, 17 links, 16 joints
Links:
- removed link base_link
- added link Body, mass 15.156; collision mesh filename=package://dog_asm2/meshes/Body.STL; visual mesh filename=package://dog_asm2/meshes/Body.STL
- link LegDownLB: geometry collision mesh filename=package://dog_asm2/meshes/LegDownLB.STL; visual mesh filename=package://dog_asm2/meshes/LegDownLB.STL
- link LegDownLF: mass 1.05169812231526 -> 1.0517; geometry collision mesh filename=package://dog_asm2/meshes/LegDownLF.STL; visual mesh filename=package://dog_asm2/meshes/LegDownLF.STL
- link LegDownRB: geometry collision mesh filename=package://dog_asm2/meshes/LegDownRB.STL; visual mesh filename=package://dog_asm2/meshes/LegDownRB.STL
- link LegDownRF: geometry collision mesh filename=package://dog_asm2/meshes/LegDownRF.STL; visual mesh filename=package://dog_asm2/meshes/LegDownRF.STL
- link LegUpLB: geometry collision mesh filename=package://dog_asm2/meshes/LegUpLB.STL; visual mesh filename=package://dog_asm2/meshes/LegUpLB.STL
- link LegUpLF: mass 1.801530833824 -> 1.8015; geometry collision mesh filename=package://dog_asm2/meshes/LegUpLF.STL; visual mesh filename=package://dog_asm2/meshes/LegUpLF.STL
- link LegUpRB: geometry collision mesh filename=package://dog_asm2/meshes/LegUpRB.STL; visual mesh filename=package://dog_asm2/meshes/LegUpRB.STL
- link LegUpRF: geometry collision mesh filename=package://dog_asm2/meshes/LegUpRF.STL; visual mesh filename=package://dog_asm2/meshes/LegUpRF.STL
- link ShoulderLB: geometry collision mesh filename=package://dog_asm2/meshes/ShoulderLB.STL; visual mesh filename=package://dog_asm2/meshes/ShoulderLB.STL
- link ShoulderLF: geometry collision mesh filename=package://dog_asm2/meshes/ShoulderLF.STL; visual mesh filename=package://dog_asm2/meshes/ShoulderLF.STL
- link ShoulderRB: mass 0.71325 -> 0.71324; geometry collision mesh filename=package://dog_asm2/meshes/ShoulderRB.STL; visual mesh filename=package://dog_asm2/meshes/ShoulderRB.STL
- link ShoulderRF: geometry collision mesh filename=package://dog_asm2/meshes/ShoulderRF.STL; visual mesh filename=package://dog_asm2/meshes/ShoulderRF.STL
- link WheelLB: geometry collision mesh filename=package://dog_asm2/meshes/WheelLB.STL; visual mesh filename=package://dog_asm2/meshes/WheelLB.STL
- link WheelLF: mass 0.327510634723198 -> 0.32751; geometry collision mesh filename=package://dog_asm2/meshes/WheelLF.STL; visual mesh filename=package://dog_asm2/meshes/WheelLF.STL
- link WheelRB: geometry collision mesh filename=package://dog_asm2/meshes/WheelRB.STL; visual mesh filename=package://dog_asm2/meshes/WheelRB.STL
- link WheelRF: geometry collision mesh filename=package://dog_asm2/meshes/WheelRF.STL; visual mesh filename=package://dog_asm2/meshes/WheelRF.STL
Joints:
- joint JLegDownLB: origin xyz=0.33 0 -0.015 rpy=0 0 -2.3761 -> xyz=0.33 0 -0.035 rpy=0 0 0
- joint JLegDownLF: origin xyz=0.33 0 -0.035 rpy=0 0 -2.4666 -> xyz=0.33 0 -0.035 rpy=0 0 0
- joint JLegDownRB: origin xyz=0.33 0 -0.015 rpy=0 0 2.1041 -> xyz=0.33 0 -0.035 rpy=0 0 0
- joint JLegDownRF: origin xyz=0.33 0 -0.015 rpy=0 0 1.9242 -> xyz=0.33 0 -0.035 rpy=0 0 0
- joint JLegUpLB: origin xyz=0.12 0 0 rpy=1.5708 -0.98423 1.5708 -> xyz=0 -0.14 0 rpy=-1.5708 0 3.1416
- joint JLegUpLF: origin xyz=0.14 0 0 rpy=-1.5708 0.92098 -1.5708 -> xyz=0 -0.14 0 rpy=-1.5708 0 3.1416
- joint JLegUpRB: origin xyz=0.12 0 0 rpy=-1.5708 -0.91233 -1.5708 -> xyz=0 -0.14 0 rpy=-1.5708 0 3.1416
- joint JLegUpRF: origin xyz=0.12 0 0 rpy=1.5708 0.69315 1.5708 -> xyz=0 -0.14 0 rpy=-1.5708 0 3.1416
- joint JShoulderLB: origin xyz=-0.29653 0.09 0.045 rpy=-1.5708 -0.012948 1.5708 -> xyz=-0.29653 0.09 0.045 rpy=3.1416 1.5708 0; parent base_link -> Body
- joint JShoulderLF: origin xyz=0.29653 0.09 0.045 rpy=1.5708 -0.12984 1.5708 -> xyz=0.29653 0.09 0.045 rpy=0 -1.5708 0; parent base_link -> Body
- joint JShoulderRB: origin xyz=-0.29653 -0.09 0.045 rpy=1.5708 0.082864 -1.5708 -> xyz=-0.29653 -0.09 0.045 rpy=3.1416 -1.5708 0; parent base_link -> Body
- joint JShoulderRF: origin xyz=0.29653 -0.09 0.045 rpy=-1.5708 0.0031802 -1.5708 -> xyz=0.29653 -0.09 0.045 rpy=0 1.5708 0; parent base_link -> Body
